File: stm32f446.kicad_pcb (KiCad board)
At the start: 2 copper layers, 42.5 x 65 mm, 61 parts, among them J1 USB_C_Receptacle_USB2.0_16P, J10 Conn_01x04_Socket, J11 Conn_01x02_Socket, J12 Conn_01x02_Socket, J13 Conn_01x04_Socket, J14 Conn_01x02_Socket, J15 Conn_01x02_Socket, J16 Conn_01x02_Socket, J17 Conn_01x02_Socket, J18 Conn_01x02_Socket, J19 Conn_01x02_Socket, J20 Conn_01x02_Socket, J3 Conn_01x03_Pin, J4 Conn_01x06_Pin, J5 Conn_01x02_Pin, J6 Conn_01x02_Pin, J7 Conn_01x02_Pin, J8 Conn_01x02_Pin, J9 Conn_01x04_Socket, SW1 SW_Push, U1 STM32F446RETx, U3 MCP1703Ax-330xxDB, U4 CH340N, Y1 ABM3B

Commit message: Update sch and pcb
Parts:
- removed J3: Conn_01x03_Pin, Connector_PinHeader_2.54mm:PinHeader_1x03_P2.54mm_Vertical
- added D10: LED, LED_SMD:LED_0603_1608Metric, F.Cu at (113.9, 123.0)
- added J2: USB_B_Micro, Connector_USB:USB_Micro-B_Amphenol_10118194-0001LF_Horizontal, F.Cu at (87.5, 63.7)
- added R16: 1k, Resistor_SMD:R_0201_0603Metric, F.Cu at (113.9, 120.3)
- added SW2: SW_SPDT, Original:SPDT_akitsuki, F.Cu at (84.1, 82.3)
- added SW3: SW_Push, Button_Switch_SMD:SW_SPST_TL3305A, F.Cu at (82.0, 136.0)
- added SW4: SW_DIP_x04, Button_Switch_THT:SW_DIP_SPSTx04_Slide_9.78x12.34mm_W7.62mm_P2.54mm, F.Cu at (95.2, 137.8)
- added U2: USBLC6-2SC6, Package_TO_SOT_SMD:SOT-23-6, F.Cu at (91.0, 76.0)
- moved J18 158.2 mm to (73.0, 86.0), turned to 0 degrees
- moved J13 130.9 mm to (73.0, 111.9)
- moved J17 113.0 mm to (127.0, 125.5)
- moved J4 98.3 mm to (85.2, 72.0)
- moved J7 95.5 mm to (73.0, 134.5)
- moved J11 95.3 mm to (73.0, 128.0)
- moved J14 93.0 mm to (73.0, 105.5)
- moved J16 91.9 mm to (73.1, 78.0)
- moved R14 90.6 mm to (117.0, 88.7), turned to 90 degrees
- moved R15 89.8 mm to (114.3, 88.7), turned to 90 degrees
- moved D8 89.8 mm to (117.0, 86.0), turned to -90 degrees
- moved J5 89.6 mm to (73.0, 63.0)
- moved D9 89.0 mm to (114.3, 86.0), turned to -90 degrees
- moved J19 87.9 mm to (73.0, 97.0), turned to 180 degrees
- moved C17 87.1 mm to (98.5, 119.0)
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Connections:
- J12 pad 1: CAN2_TX -> TIM3_CH2
- J12 pad 2: CAN2_RX -> TIM3_CH1
- U1 pad 2: FreeIO3 -> DIP2
- U1 pad 22: ADC1 -> TIM3_CH1
- U1 pad 23: ADC2 -> TIM3_CH2
- U1 pad 24: unconnected-(U1-PC4-Pad24) -> LED5
- U1 pad 26: unconnected-(U1-PB0-Pad26) -> ADC1
- U1 pad 27: unconnected-(U1-PB1-Pad27) -> ADC2
- U1 pad 28: unconnected-(U1-PB2-Pad28) -> BUTTON_INPUT
- U1 pad 29: unconnected-(U1-PB10-Pad29) -> I2C_SCL
- U1 pad 3: FreeIO4 -> DIP3
- U1 pad 33: CAN2_RX -> FreeIO4
- U1 pad 34: CAN2_TX -> FreeIO3
- U1 pad 35: unconnected-(U1-PB14-Pad35) -> FreeIO2
- U1 pad 36: unconnected-(U1-PB15-Pad36) -> FreeIO1
- U1 pad 37: Encoder_A -> UART_TX(STM)
- U1 pad 38: Encoder_B -> UART_RX(STM)
- U1 pad 4: unconnected-(U1-PC15-Pad4) -> DIP4
- U1 pad 42: UART_TX(STM) -> USB_VBUS
- U1 pad 43: UART_RX(STM) -> unconnected-(U1-PA10-Pad43)
- U1 pad 44: unconnected-(U1-PA11-Pad44) -> USB_DM
- U1 pad 45: unconnected-(U1-PA12-Pad45) -> USB_DP
- U1 pad 52: FreeIO1 -> DIP1
- U1 pad 53: FreeIO2 -> I2C_SDA
- U1 pad 54: unconnected-(U1-PD2-Pad54) -> BUTTON_3V3
- U1 pad 58: I2C_SCL -> Encoder_B
- U1 pad 59: I2C_SDA -> Encoder_A
Routing:
- net +3.3V: track 11.6 -> 84.6 mm
- net UART3_RX: track 29.9 -> 0.00 mm, vias 2 -> 0
- net SPI1_MISO: track 27.9 -> 0.00 mm, vias 2 -> 0
- net SPI1_MOSI: track 26.6 -> 0.00 mm, vias 2 -> 0
- net SWCLK: track 26.4 -> 0.00 mm
- net SWDIO: track 25.8 -> 0.00 mm, vias 1 -> 0
- net UART3_TX: track 25.3 -> 0.00 mm, vias 2 -> 0
- net NRST: track 25.2 -> 0.00 mm, vias 1 -> 0
- net CAN_TX: track 24.8 -> 0.00 mm, vias 1 -> 0
- net SWO: track 24.3 -> 0.00 mm, vias 1 -> 0
- net CAN_RX: track 22.9 -> 0.00 mm, vias 1 -> 0
- net UART_TX(STM): track 18.6 -> 0.00 mm, vias 2 -> 0
- net UART_RX(STM): track 18.3 -> 0.00 mm, vias 2 -> 0
- net SPI1_CS: track 16.1 -> 0.00 mm, vias 1 -> 0
- net ADC2: track 15.8 -> 0.00 mm, vias 1 -> 0
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Other:
- board size 42.5 x 65 mm -> 60 x 80 mm
