File: stm32f446.kicad_sch (KiCad schematic)
At the start: 61 parts, among them J1 USB_C_Receptacle_USB2.0_16P, J10 Conn_01x04_Socket, J11 Conn_01x02_Socket, J12 Conn_01x02_Socket, J13 Conn_01x04_Socket, J14 Conn_01x02_Socket, J15 Conn_01x02_Socket, J16 Conn_01x02_Socket, J17 Conn_01x02_Socket, J18 Conn_01x02_Socket, J19 Conn_01x02_Socket, J20 Conn_01x02_Socket, J3 Conn_01x03_Pin, J4 Conn_01x06_Pin, J5 Conn_01x02_Pin, J6 Conn_01x02_Pin, J7 Conn_01x02_Pin, J8 Conn_01x02_Pin, J9 Conn_01x04_Socket, SW1 SW_Push, U1 STM32F446RETx, U3 MCP1703Ax-330xxDB, U4 CH340N, Y1 ABM3B

Commit message: Update sch and pcb
Parts:
- removed J3: Conn_01x03_Pin, Connector_PinHeader_2.54mm:PinHeader_1x03_P2.54mm_Vertical, symbol Connector:Conn_01x03_Pin
- added D10: LED, LED_SMD:LED_0603_1608Metric, symbol Device:LED
- added J2: USB_B_Micro, Connector_USB:USB_Micro-B_Amphenol_10118194-0001LF_Horizontal, symbol Connector:USB_B_Micro
- added R16: 1k, Resistor_SMD:R_0201_0603Metric, symbol Device:R
- added SW2: SW_SPDT, Original:SPDT_akitsuki, symbol Switch:SW_SPDT
- added SW3: SW_Push, Button_Switch_SMD:SW_SPST_TL3305A, symbol Switch:SW_Push
- added SW4: SW_DIP_x04, Button_Switch_THT:SW_DIP_SPSTx04_Slide_9.78x12.34mm_W7.62mm_P2.54mm, symbol Switch:SW_DIP_x04
- added U2: USBLC6-2SC6, Package_TO_SOT_SMD:SOT-23-6, symbol Power_Protection:USBLC6-2SC6
Connections:
- net +3.3V: now also SW2.1 (A)
- net ADC1: now also U1.26 (PB0); no longer U1.22 (PA6)
- net ADC2: now also U1.27 (PB1); no longer U1.23 (PA7)
- net BOOT0: now also SW2.2 (B)
- net Encoder_A: now also U1.59 (PB7); no longer U1.37 (PC6)
- net Encoder_B: now also U1.58 (PB6); no longer U1.38 (PC7)
- net FreeIO1: now also U1.36 (PB15); no longer U1.52 (PC11)
- net FreeIO2: now also U1.35 (PB14); no longer U1.53 (PC12)
- net FreeIO3: now also U1.34 (PB13); no longer U1.2 (PC13)
- net FreeIO4: now also U1.33 (PB12); no longer U1.3 (PC14)
- net GND: now also D10.1 (K), J2.5 (GND), J2.SH (Shield), U2.2 (GND)
- net I2C_SCL: now also U1.29 (PB10); no longer U1.58 (PB6)
- net I2C_SDA: now also U1.53 (PC12); no longer U1.59 (PB7)
- net UART_RX(STM): now also U1.38 (PC7); no longer U1.43 (PA10)
- net UART_TX(STM): now also U1.37 (PC6); no longer U1.42 (PA9)
- net at R1.2: now also SW2.3 (C)
- net LED5: now reaches U1.24 (PC4)
- net LED5: now also R16.2
- net BUTTON_INPUT: now reaches U1.28 (PB2)
- net BUTTON_INPUT: now also SW3.2
- net DIP4: now reaches U1.4 (PC15)
- net DIP4: now also SW4.8
- net USB_DM: now reaches U1.44 (PA11)
- net USB_DM: now also U2.6 (I/O1)
- net USB_DP: now reaches U1.45 (PA12)
- net USB_DP: now also U2.4 (I/O2)
- net BUTTON_3V3: now reaches U1.54 (PD2)
- net BUTTON_3V3: now also SW3.1, SW4.1, SW4.2, SW4.3, SW4.4
- net CAN2_RX renamed TIM3_CH1
- net TIM3_CH1: now also U1.22 (PA6); no longer U1.33 (PB12)
- net CAN2_TX renamed TIM3_CH2
- net TIM3_CH2: now also U1.23 (PA7); no longer U1.34 (PB13)
- new net: D10.2 (A), R16.1
- new net: J2.2 (D-), U2.3 (I/O2)
- new net: J2.3 (D+), U2.1 (I/O1)
- new net +5VA: J2.1 (VBUS), U1.42 (PA9), U2.5 (VBUS)
- new net DIP1: SW4.5, U1.52 (PC11)
- new net DIP2: SW4.6, U1.2 (PC13)
- new net DIP3: SW4.7, U1.3 (PC14)
- no-connect marks 16 -> 7
Other:
- moved on the sheet: D4, D5, D6, D7, D8, D9, J10, J11, J13, J14, J15, J19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
